File: VCO/vco.sch (KiCad schematic (older format))
At the start: 50 parts

Commit message: VCO update
vco pcb, gerbers and bom updated
Parts:
- added C10: .002uF, Capacitors_SMD:C_0805, symbol CP1
- added C11: 10pF, Capacitors_SMD:C_0805, symbol CP1_Small
- added C12, C13: .1uF, Capacitors_SMD:C_0805, symbol CP1_Small
- added C14, C15: 1uF, Capacitors_SMD:C_0805, symbol CP1
- added C4, C9: .1uF, Capacitors_SMD:C_0805, symbol CP1
- added D3, D4, D5, D6, D7, D8: D, Diodes_SMD:D_MiniMELF, symbol D
- added R22, R34, R44, R45: 100K, Resistors_SMD:R_0805, symbol R
- added R26, R29, R30, R35, R36, R47: 10K, Resistors_SMD:R_0805, symbol R
- added R27: 470K, Resistors_SMD:R_0805, symbol R
- added R28: 47K, Resistors_SMD:R_0805, symbol R
- added R31, R33, R40, R41: 1K, Resistors_SMD:R_0805, symbol R
- added R32: 20k, Resistors_SMD:R_0805, symbol R
- added R37: 1M, Resistors_SMD:R_0805, symbol R
- added R38, R39: 20K, Resistors_SMD:R_0805, symbol R
- added R42, R48: 4.7K, Resistors_SMD:R_0805, symbol R
- added R43: 130K, Resistors_SMD:R_0805, symbol R
- added R46: 10M, Resistors_SMD:R_0805, symbol R
- added R49: 3K, Resistors_SMD:R_0805_HandSoldering, symbol R
- added RV10: 100K, Potentiometers:Potentiometer_Alps_RK09K_Horizontal, symbol POT
- added RV4: 10K, Potentiometers:Potentiometer_Trimmer_Bourns_3214W, symbol POT-RESCUE-vco
- added RV6, RV7: 100K, Potentiometers:Potentiometer_Trimmer_Bourns_3214W, symbol POT
- added RV8: 10K, Potentiometers:Potentiometer_Trimmer_Bourns_3214X, symbol POT-RESCUE-vco
- added RV9: 1M, Potentiometers:Potentiometer_Trimmer_Bourns_3214W, symbol POT
- added U1: LM13700, Housings_SOIC:SOIC-16_3.9x9.9mm_Pitch1.27mm, symbol LM13700
- added U4: TL074, Housings_SOIC:SOIC-14_3.9x8.7mm_Pitch1.27mm, symbol TL074
- added U6: TL072, Housings_SOIC:SOIC-8_3.9x4.9mm_Pitch1.27mm, symbol TL072
- added U7: TL071, Housings_SOIC:SOIC-8_3.9x4.9mm_Pitch1.27mm, symbol TL071
- C1, C3, C7: renamed from C?; footprint (none) -> Capacitors_SMD:C_0603
- C2, C5, C6: renamed from C?; footprint (none) -> Capacitors_SMD:C_0805
- C8: renamed from C?; value CP1 -> 100pF; footprint (none) -> Capacitors_SMD:C_0603
- D1, D2: renamed from D?; footprint (none) -> Diodes_SMD:D_MiniMELF
- Q1: renamed from Q?; footprint (none) -> TO_SOT_Packages_SMD:SOT-23
- R1, R10, R11, R12, R13, R14, R15, R16, R17, R18, R19, R2, R20, R21, R23, R24, R25, R3, R4, R5, R6, R7, R8, R9: renamed from R?; footprint (none) -> Resistors_SMD:R_0805
- RV1, RV2: renamed from RV?; footprint (none) -> Potentiometers:Potentiometer_Alps_RK09K_Horizontal; symbol POT -> POT-RESCUE-vco
- RV3, RV5: renamed from RV?; footprint (none) -> Potentiometers:Potentiometer_Trimmer_Bourns_3214W; symbol POT -> POT-RESCUE-vco
- TH1, TH2: renamed from TH?; footprint (none) -> Resistors_SMD:R_1206
- U2, U3, U5: renamed from U?; footprint (none) -> Housings_SOIC:SOIC-8_3.9x4.9mm_Pitch1.27mm
- W1, W2, W3, W4: renamed from W?; footprint (none) -> Wire_Pads:SolderWirePad_single_2mmDrill
Connections:
- net +12V: now also C12.1, R22.1, R35.1, R37.1, RV6.1, RV9.1, U1.11 (V+), U1.11 (V+), U4.4 (V+), U4.4 (V+), U4.4 (V+), U4.4 (V+), U6.8 (V+), U6.8 (V+), U7.7 (V+)
- net -12V: now also C10.2, C13.1, R38.1, R42.1, RV6.3, U1.6 (V-), U1.6 (V-), U4.11 (V-), U4.11 (V-), U4.11 (V-), U4.11 (V-), U6.4 (V-), U6.4 (V-), U7.4 (V-)
- net GND: now also C12.2, C13.2, C14.2, C15.1, C4.2, C9.2, R31.2, R43.1, R45.2, R49.2, RV4.3, RV8.3, U1.13 (INPUT(-)), U1.14 (INPUT(+)), U1.4 (INPUT(-)), U4.10 (+), U4.3 (+)
- net RAW: now also R26.2
- net at D1.2 (A), U5.2 (B): now also RV3.2; no longer RV3.1
- net at C1.2, TH2.1, U3.1: now also RV3.1
- net at C7.2, R16.1, U3.7: now also RV5.3; no longer RV5.2
- net at RV2.1: now also R10.2; no longer R3.2
- net at RV2.2: now also R3.2; no longer R2.1
- net at RV2.3: now also R2.1
- net at RV1.1: now also R9.2; no longer R4.2
- net at RV1.2: now also R4.2; no longer R1.1
- net at RV1.3: now also R1.1
- net at R11.1: now also RV3.3; no longer RV3.2
- net at R14.1, RV5.1: now also RV5.2
- new net: C4.1, RV4.2, U4.5 (+)
- new net: R26.1, R28.2, U4.6 (-)
- new net: D4.2 (A), R28.1, R29.1, U4.7
- new net: R34.2, U1.1 (AMP_BIAS_INPUT)
- new net: R27.2, R31.1, R32.2, U1.3 (INPUT(+))
- new net: R37.2, R43.2, U1.5 (OUTPUT), U1.7 (BUFFER_INPUT)
- new net: R41.2, R42.2, U1.8 (BUFFER_OUTPUT)
- new net: D3.2 (A), D5.2 (A), D6.1 (K), R30.1, R33.2, R44.2, U4.8
- new net: R29.2, R30.2, U4.9 (-)
- new net: R22.2, RV4.1
- new net: U4.1, U4.2 (-)
- new net: C9.1, RV8.2, U4.12 (+)
- new net: R36.1, R39.2, U4.13 (-)
- new net: R35.2, RV8.1
- new net: C10.1, D3.1 (K), D4.1 (K), R36.2, R38.2
- new net: R27.1, RV6.2
- new net: R32.1, RV7.2, RV7.3
- new net: R34.1, RV9.2, RV9.3
- new net: RV10.1, U6.1, U6.2 (-)
- new net: C14.1, D5.1 (K), U6.3 (+)
- new net: C15.2, D8.2 (A), U6.5 (+)
- new net: RV10.3, U6.6 (-), U6.7
- new net: D6.2 (A), D7.1 (K)
- new net: D7.2 (A), D8.1 (K)
- new net: C11.1, R44.1, R46.2, U7.3 (+)
- new net: C11.2, R46.1, R48.1, U7.6
- new net: R47.2, RV10.2
- new net PWM: R45.1, R47.1, U7.2 (-)
- new net RMP: R33.1
- new net SIN: R41.1
- new net SINSHAPER: R39.1, R40.2, RV7.1, U4.14
- new net SQR: R48.2, R49.1
- new net TRI: R40.1
Other:
- note added: "PANEL MOUNTED\n"
- note added: "Pulse Width Adj.\n"
- note added: "RAMP OFFSET TRIM"
- note added: "Sine Bias Trim\n"
- note added: "Sine Level Trim\n"
- note added: "Sine Shape Trim\n"
- note added: "TRAINGLE OFFSET TRIM"

Commit message: Changed Pot
Trimmer potentiometer was too expensive, updated pcb and gerbers for cheaper trimmer pot
Parts:
- RV3, RV4, RV5, RV6, RV7, RV9: footprint Potentiometers:Potentiometer_Trimmer_Bourns_3214W -> Potentiometers:Potentiometer_Trimmer-EVM3E
- RV8: footprint Potentiometers:Potentiometer_Trimmer_Bourns_3214X -> Potentiometers:Potentiometer_Trimmer-EVM3E
Changed lines of the file:
@@
 EESchema Schematic File Version 2
-LIBS:vco-rescue
 LIBS:power
 LIBS:device
@@
 F 0 "RV3" H 2700 2570 50  0000 C CNN
 F 1 "100" H 2700 2650 50  0000 C CNN
-F 2 "Potentiometers:Potentiometer_Trimmer_Bourns_3214W" H 2700 2650 50  0001 C CNN
+F 2 "Potentiometers:Potentiometer_Trimmer-EVM3E" H 2700 2650 50  0001 C CNN
 F 3 "" H 2700 2650 50  0000 C CNN
 	1    2700 2650
@@
 F 0 "RV5" H 4700 1870 50  0000 C CNN
 F 1 "100K" H 4700 1950 50  0000 C CNN
-F 2 "Potentiometers:Potentiometer_Trimmer_Bourns_3214W" H 4700 1950 50  0001 C CNN
+F 2 "Potentiometers:Potentiometer_Trimmer-EVM3E" H 4700 1950 50  0001 C CNN
 F 3 "" H 4700 1950 50  0000 C CNN
 	1    4700 1950
@@
 F 0 "RV4" H 4550 870 50  0000 C CNN
 F 1 "10K" H 4550 950 50  0000 C CNN
-F 2 "Potentiometers:Potentiometer_Trimmer_Bourns_3214W" H 4550 950 50  0001 C CNN
+F 2 "Potentiometers:Potentiometer_Trimmer-EVM3E" H 4550 950 50  0001 C CNN
 F 3 "" H 4550 950 50  0000 C CNN
 	1    4550 950
@@
 F 0 "RV8" H 6600 720 50  0000 C CNN
 F 1 "10K" H 6600 800 50  0000 C CNN
-F 2 "Potentiometers:Potentiometer_Trimmer_Bourns_3214X" H 6600 800 50  0001 C CNN
+F 2 "Potentiometers:Potentiometer_Trimmer-EVM3E" H 6600 800 50  0001 C CNN
 F 3 "" H 6600 800 50  0000 C CNN
 	1    6600 800
@@
 F 0 "RV6" V 5425 4900 50  0000 C CNN
 F 1 "100K" V 5500 4900 50  0000 C CNN
-F 2 "Potentiometers:Potentiometer_Trimmer_Bourns_3214W" H 5600 4900 50  0001 C CNN
+F 2 "Potentiometers:Potentiometer_Trimmer-EVM3E" H 5600 4900 50  0001 C CNN
 F 3 "" H 5600 4900 50  0001 C CNN
 	1    5600 4900
@@
 F 0 "RV7" V 6075 4600 50  0000 C CNN
 F 1 "100K" V 6150 4600 50  0000 C CNN
-F 2 "Potentiometers:Potentiometer_Trimmer_Bourns_3214W" H 6250 4600 50  0001 C CNN
+F 2 "Potentiometers:Potentiometer_Trimmer-EVM3E" H 6250 4600 50  0001 C CNN
 F 3 "" H 6250 4600 50  0001 C CNN
 	1    6250 4600
@@
 F 0 "RV9" V 6675 5000 50  0000 C CNN
 F 1 "1M" V 6750 5000 50  0000 C CNN
-F 2 "Potentiometers:Potentiometer_Trimmer_Bourns_3214W" H 6850 5000 50  0001 C CNN
+F 2 "Potentiometers:Potentiometer_Trimmer-EVM3E" H 6850 5000 50  0001 C CNN
 F 3 "" H 6850 5000 50  0001 C CNN
 	1    6850 5000
